Commit message: initial modi

File: urdf/spotrobot.urdf (robot description, URDF)
Before this commit: robot quadruped_leg, 17 links, 16 joints
Links:
- link base_link: mass None -> 1; geometry collision box size=0.3 0.1 0.02; visual box size=0.3 0.1 0.02
- link body1_link: mass None -> 1; geometry collision cylinder length=0.035 radius=0.005; visual box size=0.03 0.03 0.02
- link body2_link: mass None -> 1; geometry collision cylinder length=0.035 radius=0.005; visual box size=0.02 0.01 0.05
- link body3_link: mass None -> 1; geometry collision cylinder length=0.035 radius=0.005; visual box size=0.01 0.01 0.1
- link shank_link_back: mass None -> 1; geometry collision cylinder length=0.035 radius=0.005; visual cylinder length=0.05 radius=0.005
- link shank_link_back1: mass None -> 1; geometry collision cylinder length=0.035 radius=0.005; visual cylinder length=0.05 radius=0.005
- link shank_link_front: mass None -> 1; geometry collision cylinder length=0.035 radius=0.005; visual cylinder length=0.05 radius=0.005
- link shank_link_front1: mass None -> 1; geometry collision cylinder length=0.035 radius=0.005; visual cylinder length=0.05 radius=0.005
- link shoulder_link_back: mass None -> 1; geometry collision cylinder length=0.035 radius=0.005; visual cylinder length=0.035 radius=0.005
- link shoulder_link_back1: mass None -> 1; geometry collision cylinder length=0.035 radius=0.005; visual cylinder length=0.035 radius=0.005
- link shoulder_link_front: mass None -> 1; geometry collision cylinder length=0.035 radius=0.005; visual cylinder length=0.035 radius=0.005
- link shoulder_link_front1: mass None -> 1; geometry collision cylinder length=0.035 radius=0.005; visual cylinder length=0.035 radius=0.005
- link thigh_link_back: mass None -> 1; geometry collision cylinder length=0.035 radius=0.005; visual cylinder length=0.045 radius=0.01
- link thigh_link_back1: mass None -> 1; geometry collision cylinder length=0.035 radius=0.005; visual cylinder length=0.045 radius=0.01
- link thigh_link_front: mass None -> 1; geometry collision cylinder length=0.035 radius=0.005; visual cylinder length=0.045 radius=0.01
- link thigh_link_front1: mass None -> 1; geometry collision cylinder length=0.035 radius=0.005; visual cylinder length=0.045 radius=0.01

Commit message: controller working

File: urdf/spotrobot.urdf (robot description, URDF)
Before this commit: robot quadruped_leg, 10 links, 9 joints
Joints:
- joint body1_joint: limit lower=-0.03 upper=0.0 effort=0 velocity=0 -> (none); type prismatic -> fixed
