Commit message: updated wtout shoulder

File: urdf/spotmini.urdf (robot description, URDF)
Before this commit: robot quadruped_leg, 17 links, 16 joints
Links:
- removed link body2_link
- removed link body3_link
- removed link body4_link
- removed link shoulder_link_back
- removed link shoulder_link_back1
- removed link shoulder_link_front
- removed link shoulder_link_front1
Joints:
- removed joint body2_joint
- removed joint body3_joint
- removed joint body4_joint
- removed joint shoulder_joint_back
- removed joint shoulder_joint_back1
- removed joint shoulder_joint_front
- removed joint shoulder_joint_front1
- joint elbow_joint_back: origin xyz=0 -0.025 -0.005 -> xyz=-0.145 -0.045 -0.01; parent shoulder_link_back -> base_link
- joint elbow_joint_back1: origin xyz=0 -0.0125 -0.005 -> xyz=-0.145 0.045 -0.01; parent shoulder_link_back1 -> base_link
- joint elbow_joint_front: origin xyz=0 -0.025 -0.005 -> xyz=0.145 -0.045 -0.01; parent shoulder_link_front -> base_link
- joint elbow_joint_front1: origin xyz=0.0 -0.02 -0.005 -> xyz=0.145 0.045 -0.01; parent shoulder_link_front1 -> base_link

Commit message: controller added

File: urdf/spotmini.urdf (robot description, URDF)
Before this commit: robot spot mini, 10 links, 9 joints
Links:
- link body1_link: mass None -> 1; geometry collision box size=0.03 0.03 0.02; visual box size=0.03 0.03 0.02
- link shank_link_back: mass None -> 1; geometry collision cylinder length=0.05 radius=0.005; visual cylinder length=0.05 radius=0.005
- link shank_link_back1: mass None -> 1; geometry collision cylinder length=0.05 radius=0.005; visual cylinder length=0.05 radius=0.005
- link shank_link_front: mass None -> 1; geometry collision cylinder length=0.05 radius=0.005; visual cylinder length=0.05 radius=0.005
- link shank_link_front1: mass None -> 1; geometry collision cylinder length=0.05 radius=0.005; visual cylinder length=0.05 radius=0.005
- link thigh_link_back: mass None -> 1; geometry collision cylinder length=0.045 radius=0.01; visual cylinder length=0.045 radius=0.01
- link thigh_link_back1: mass None -> 1; geometry collision cylinder length=0.045 radius=0.01; visual cylinder length=0.045 radius=0.01
- link thigh_link_front: mass None -> 1; geometry collision cylinder length=0.045 radius=0.01; visual cylinder length=0.045 radius=0.01
- link thigh_link_front1: mass None -> 1; geometry collision cylinder length=0.045 radius=0.01; visual cylinder length=0.045 radius=0.01
Joints:
- joint elbow_joint_back: limit lower=-1.57075 upper=1.57075 effort=1000.0 velocity=0.5 -> lower=-1.57075 upper=1.57075 effort=5.0 velocity=0.5
- joint elbow_joint_back1: limit lower=-1.57075 upper=1.57075 effort=1000.0 velocity=0.5 -> lower=-1.57075 upper=1.57075 effort=5.0 velocity=0.5
- joint elbow_joint_front: limit lower=-1.57075 upper=1.57075 effort=1000.0 velocity=0.5 -> lower=-1.57075 upper=1.57075 effort=5.0 velocity=0.5
- joint elbow_joint_front1: limit lower=-1.57075 upper=1.57075 effort=1000.0 velocity=0.5 -> lower=-0.52366 upper=0.52366 effort=1.0 velocity=0.5
- joint wrist_joint_back: limit lower=-1.57075 upper=1.57075 effort=1000.0 velocity=0.5 -> lower=-1.57075 upper=1.57075 effort=5.0 velocity=0.5
- joint wrist_joint_back1: limit lower=-1.57075 upper=1.57075 effort=1000.0 velocity=0.5 -> lower=-1.57075 upper=1.57075 effort=5.0 velocity=0.5
- joint wrist_joint_front: limit lower=-1.57075 upper=1.57075 effort=1000.0 velocity=0.5 -> lower=-1.57075 upper=1.57075 effort=5.0 velocity=0.5
- joint wrist_joint_front1: limit lower=-1.57075 upper=1.57075 effort=1000.0 velocity=0.5 -> lower=-1.57075 upper=1.57075 effort=5.0 velocity=0.5

Commit message: displayed in gazebo

File: urdf/spotmini.urdf (robot description, URDF)
Before this commit: robot spot mini, 10 links, 9 joints
Links:
- added link body2_link; visual box size=0.02 0.01 0.05
- added link body3_link; visual box size=0.01 0.01 0.1
- added link body4_link; visual box size=0.01 0.01 0.1
- added link shoulder_link_back; visual cylinder length=0.035 radius=0.005
- added link shoulder_link_back1; visual cylinder length=0.035 radius=0.005
- added link shoulder_link_front; visual cylinder length=0.035 radius=0.005
- added link shoulder_link_front1; visual cylinder length=0.035 radius=0.005
- link body1_link: mass 1 -> None; geometry visual box size=0.03 0.03 0.02
- link shank_link_back: mass 1 -> None; geometry visual cylinder length=0.05 radius=0.005
- link shank_link_back1: mass 1 -> None; geometry visual cylinder length=0.05 radius=0.005
- link shank_link_front: mass 1 -> None; geometry visual cylinder length=0.05 radius=0.005
- link shank_link_front1: mass 1 -> None; geometry visual cylinder length=0.05 radius=0.005
- link thigh_link_back: mass 1 -> None; geometry visual cylinder length=0.045 radius=0.01
- link thigh_link_back1: mass 1 -> None; geometry visual cylinder length=0.045 radius=0.01
- link thigh_link_front: mass 1 -> None; geometry visual cylinder length=0.045 radius=0.01
- link thigh_link_front1: mass 1 -> None; geometry visual cylinder length=0.045 radius=0.01
Joints:
- added joint body2_joint: type revolute, parent body1_link, child body2_link, origin xyz=0 0 0.02 rpy=0 0 1.57, limit lower=-0.523 upper=0.523 effort=0 velocity=0
- added joint body3_joint: type revolute, parent body2_link, child body3_link, origin xyz=0 0 0.05 rpy=0 0 0, limit lower=-1.5 upper=1.5 effort=0 velocity=0
- added joint body4_joint: type revolute, parent body3_link, child body4_link, origin xyz=0 0 0.1 rpy=0 0 0, limit lower=-1.5 upper=1.5 effort=0 velocity=0
- added joint shoulder_joint_back: type fixed, parent base_link, child shoulder_link_back, origin xyz=-0.145 -0.015 -0.015, axis 1 0 0, limit lower=-1.57075 upper=1.57075 effort=1000.0 velocity=0.5
- added joint shoulder_joint_back1: type fixed, parent base_link, child shoulder_link_back1, origin xyz=-0.145 0.050 -0.015, axis 1 0 0, limit lower=-1.57075 upper=1.57075 effort=1000.0 velocity=0.5
- added joint shoulder_joint_front: type fixed, parent base_link, child shoulder_link_front, origin xyz=0.145 -0.015 -0.015, axis 1 0 0, limit lower=-1.57075 upper=1.57075 effort=1000.0 velocity=0.5
- added joint shoulder_joint_front1: type fixed, parent base_link, child shoulder_link_front1, origin xyz=0.145 0.05 -0.015, axis 1 0 0, limit lower=-1.57075 upper=1.57075 effort=1000.0 velocity=0.5
- joint elbow_joint_back: limit lower=-1.57075 upper=1.57075 effort=5.0 velocity=0.5 -> lower=-1.57075 upper=1.57075 effort=1000.0 velocity=0.5; origin xyz=-0.145 -0.045 -0.01 -> xyz=0 -0.025 -0.005; parent base_link -> shoulder_link_back
- joint elbow_joint_back1: limit lower=-1.57075 upper=1.57075 effort=5.0 velocity=0.5 -> lower=-1.57075 upper=1.57075 effort=1000.0 velocity=0.5; origin xyz=-0.145 0.045 -0.01 -> xyz=0 -0.0125 -0.005; parent base_link -> shoulder_link_back1
- joint elbow_joint_front: limit lower=-1.57075 upper=1.57075 effort=5.0 velocity=0.5 -> lower=-1.57075 upper=1.57075 effort=1000.0 velocity=0.5; origin xyz=0.145 -0.045 -0.01 -> xyz=0 -0.025 -0.005; parent base_link -> shoulder_link_front
- joint elbow_joint_front1: limit lower=-0.52366 upper=0.52366 effort=1.0 velocity=0.5 -> lower=-1.57075 upper=1.57075 effort=1000.0 velocity=0.5; origin xyz=0.145 0.045 -0.01 -> xyz=0.0 -0.02 -0.005; parent base_link -> shoulder_link_front1
- joint wrist_joint_back: limit lower=-1.57075 upper=1.57075 effort=5.0 velocity=0.5 -> lower=-1.57075 upper=1.57075 effort=1000.0 velocity=0.5
- joint wrist_joint_back1: limit lower=-1.57075 upper=1.57075 effort=5.0 velocity=0.5 -> lower=-1.57075 upper=1.57075 effort=1000.0 velocity=0.5
- joint wrist_joint_front: limit lower=-1.57075 upper=1.57075 effort=5.0 velocity=0.5 -> lower=-1.57075 upper=1.57075 effort=1000.0 velocity=0.5
- joint wrist_joint_front1: limit lower=-1.57075 upper=1.57075 effort=5.0 velocity=0.5 -> lower=-1.57075 upper=1.57075 effort=1000.0 velocity=0.5

File: urdf/spotrobot.urdf (robot description, URDF)
Before this commit: robot quadruped_leg, 14 links, 13 joints
Links:
- removed link shoulder_link_back
- removed link shoulder_link_back1
- removed link shoulder_link_front
- removed link shoulder_link_front1
Joints:
- removed joint shoulder_joint_back
- removed joint shoulder_joint_back1
- removed joint shoulder_joint_front
- removed joint shoulder_joint_front1
- joint elbow_joint_back: origin xyz=0 -0.025 -0.005 -> xyz=-0.145 -0.045 -0.01; parent shoulder_link_back -> base_link
- joint elbow_joint_back1: origin xyz=0 -0.0125 -0.005 -> xyz=-0.145 0.045 -0.01; parent shoulder_link_back1 -> base_link
- joint elbow_joint_front: origin xyz=0 -0.025 -0.005 -> xyz=0.145 -0.045 -0.01; parent shoulder_link_front -> base_link
- joint elbow_joint_front1: origin xyz=0.0 -0.02 -0.005 -> xyz=0.145 0.045 -0.01; parent shoulder_link_front1 -> base_link

Commit message: controller added

File: urdf/spotmini.urdf (robot description, URDF)
Before this commit: robot quadruped_leg, 17 links, 16 joints
Links:
- removed link shoulder_link_back
- removed link shoulder_link_back1
- removed link shoulder_link_front
- removed link shoulder_link_front1
- added link imu_sensor_link, mass 0.001; collision box size=0.005 0.005 0.005; visual box size=0.005 0.005 0.005
- link base_link: mass None -> 1; geometry collision box size=0.3 0.1 0.02; visual box size=0.3 0.1 0.02
- link body1_link: mass None -> 1; geometry collision cylinder length=0.035 radius=0.005; visual box size=0.03 0.03 0.02
- link body2_link: mass None -> 1; geometry collision box size=0.02 0.01 0.05; visual box size=0.02 0.01 0.05
- link body3_link: mass None -> 1; geometry collision box size=0.01 0.01 0.1; visual box size=0.01 0.01 0.1
- link body4_link: mass None -> 1; geometry collision box size=0.01 0.01 0.1; visual box size=0.01 0.01 0.1
- link shank_link_back: mass None -> 1; geometry collision cylinder length=0.05 radius=0.005; visual cylinder length=0.05 radius=0.005
- link shank_link_back1: mass None -> 1; geometry collision cylinder length=0.05 radius=0.005; visual cylinder length=0.05 radius=0.005
- link shank_link_front: mass None -> 1; geometry collision cylinder length=0.05 radius=0.005; visual cylinder length=0.05 radius=0.005
- link shank_link_front1: mass None -> 1; geometry collision cylinder length=0.05 radius=0.005; visual cylinder length=0.05 radius=0.005
- link thigh_link_back: mass None -> 1; geometry collision cylinder length=0.045 radius=0.01; visual cylinder length=0.045 radius=0.01
- link thigh_link_back1: mass None -> 1; geometry collision cylinder length=0.045 radius=0.01; visual cylinder length=0.045 radius=0.01
- link thigh_link_front: mass None -> 1; geometry collision cylinder length=0.045 radius=0.01; visual cylinder length=0.045 radius=0.01
- link thigh_link_front1: mass None -> 1; geometry collision cylinder length=0.045 radius=0.01; visual cylinder length=0.045 radius=0.01
Joints:
- removed joint shoulder_joint_back
- removed joint shoulder_joint_back1
- removed joint shoulder_joint_front
- removed joint shoulder_joint_front1
- added joint imu_sensor_joint: type fixed, parent body4_link, child imu_sensor_link, origin xyz=0 0.0085 0.09 rpy=0 0 0, axis 0 0 1
- joint body1_joint: limit lower=-0.03 upper=0.0 effort=0 velocity=0 -> (none); type prismatic -> fixed
- joint body2_joint: limit lower=-0.523 upper=0.523 effort=0 velocity=0 -> lower=0.32 upper=0.7 effort=10 velocity=1
- joint body3_joint: limit lower=-1.5 upper=1.5 effort=0 velocity=0 -> lower=-1.5 upper=1.5 effort=10 velocity=1
- joint body4_joint: limit lower=-1.5 upper=1.5 effort=0 velocity=0 -> lower=-0.39 upper=0.39 effort=10.0 velocity=1
- joint elbow_joint_back: limit lower=-1.57075 upper=1.57075 effort=1000.0 velocity=0.5 -> lower=-0.39 upper=0.39 effort=10.0 velocity=1.0; origin xyz=0 -0.025 -0.005 -> xyz=-0.145 -0.045 -0.01; parent shoulder_link_back -> base_link
- joint elbow_joint_back1: limit lower=-1.57075 upper=1.57075 effort=1000.0 velocity=0.5 -> lower=-0.39 upper=0.39 effort=10.0 velocity=1.0; origin xyz=0 -0.0125 -0.005 -> xyz=-0.145 0.045 -0.01; parent shoulder_link_back1 -> base_link
- joint elbow_joint_front: limit lower=-1.57075 upper=1.57075 effort=1000.0 velocity=0.5 -> lower=-0.39 upper=0.39 effort=10.0 velocity=1.0; origin xyz=0 -0.025 -0.005 -> xyz=0.145 -0.045 -0.01; parent shoulder_link_front -> base_link
- joint elbow_joint_front1: limit lower=-1.57075 upper=1.57075 effort=1000.0 velocity=0.5 -> lower=-1.57075 upper=1.57075 effort=10.0 velocity=1.0; origin xyz=0.0 -0.02 -0.005 -> xyz=0.145 0.045 -0.01; parent shoulder_link_front1 -> base_link
- joint wrist_joint_back: limit lower=-1.57075 upper=1.57075 effort=1000.0 velocity=0.5 -> lower=-0.39 upper=0.39 effort=10.0 velocity=1.0
- joint wrist_joint_back1: limit lower=-1.57075 upper=1.57075 effort=1000.0 velocity=0.5 -> effort=10.0 velocity=1.0
- joint wrist_joint_front: limit lower=-1.57075 upper=1.57075 effort=1000.0 velocity=0.5 -> lower=-0.39 upper=0.40 effort=10.0 velocity=1.0
- joint wrist_joint_front1: limit lower=-1.57075 upper=1.57075 effort=1000.0 velocity=0.5 -> lower=-0.39 upper=0.39 effort=1.0 velocity=1

File: urdf/spotrobot.urdf (robot description, URDF)
Before this commit: robot quadruped_leg, 10 links, 9 joints
Links:
- removed link body1_link
- link base_link: mass 1 -> 2
- link shank_link_back: geometry collision cylinder length=0.05 radius=0.005; visual cylinder length=0.05 radius=0.005
- link shank_link_back1: geometry collision cylinder length=0.05 radius=0.005; visual cylinder length=0.05 radius=0.005
- link shank_link_front: geometry collision cylinder length=0.05 radius=0.005; visual cylinder length=0.05 radius=0.005
- link shank_link_front1: geometry collision cylinder length=0.05 radius=0.005; visual cylinder length=0.05 radius=0.005
- link thigh_link_back: geometry collision cylinder length=0.045 radius=0.01; visual cylinder length=0.045 radius=0.01
- link thigh_link_back1: geometry collision cylinder length=0.045 radius=0.01; visual cylinder length=0.045 radius=0.01
- link thigh_link_front: geometry collision cylinder length=0.045 radius=0.01; visual cylinder length=0.045 radius=0.01
- link thigh_link_front1: geometry collision cylinder length=0.045 radius=0.01; visual cylinder length=0.045 radius=0.01
Joints:
- removed joint body1_joint
- joint elbow_joint_front: limit lower=-1.57075 upper=1.57075 effort=1000.0 velocity=0.5 -> (none); type revolute -> fixed
- joint elbow_joint_front1: limit lower=-1.57075 upper=1.57075 effort=1000.0 velocity=0.5 -> lower=-0.2678 upper=0.2679 effort=1000.0 velocity=5
- joint wrist_joint_front: limit lower=-1.57075 upper=1.57075 effort=1000.0 velocity=0.5 -> lower=-0.2678 upper=0.2679 effort=1000.0 velocity=0.5
- joint wrist_joint_front1: limit lower=-1.57075 upper=1.57075 effort=1000.0 velocity=0.5 -> lower=-0.2678 upper=0.2679 effort=1000.0 velocity=5

Commit message: image update

File: urdf/spotmini.urdf (robot description, URDF)
Before this commit: robot quadruped_leg, 14 links, 13 joints
Joints:
- joint wrist_joint_back1: limit effort=10.0 velocity=1.0 -> lower=-0.39 upper=0.39 effort=10.0 velocity=1.0

Commit message: camera link added

File: urdf/spotmini.urdf (robot description, URDF)
Before this commit: robot quadruped_leg, 14 links, 13 joints
Links:
- removed link imu_sensor_link
- added link camera_link, mass 0.001; collision box size=0.01 0.01 0.01; visual box size=0.01 0.01 0.01
Joints:
- joint imu_sensor_joint: child imu_sensor_link -> camera_link; origin xyz=0 0.0085 0.09 rpy=0 0 0 -> xyz=0.0 -0.008 0.095 rpy=0 0 0
